File: PG-Pedal-1/12-Carrier-Board/pcbway/pg1-carrier.kicad_pcb (KiCad board)
At the start: 2 copper layers, 111 x 58.2 mm, 100 parts, among them J1 in, J10 seed3 + 9v, J19 pg-hp, J2 out, J20 pg-line, J21 expansion, J22 fx loop, U1 AMS1117-5.0, U10 TPA6139A2, U11 TLV9062, U12 TLV9062, U2 XC6206P332MR, U3 B0505S-1WR3, U4 ISO7741, U5 ISO1540, U7 XC6206P332MR, U8 TLV9062, U9 TLV320AIC3204

Commit message: Carrier: simulation found the input 3.2 kHz low-pass (C31/C41 not fitted); part labels; firmware input gain; plugin face fixed
Co-Authored-By: Claude Opus 5.5 <noreply@anthropic.com>
Other:
- board text added: "3V3 REG"
- board text added: "5V REG"
- board text added: "AIC3204"
- board text added: "B0505S"
- board text added: "B5819"
- board text added: "ISO1540"
- board text added: "ISO7741"
- board text added: "PIN 1"
- board text added: "PSM712"
- board text added: "PTC"
- board text added: "TLV9062"
- board text added: "TPA6139"
Changed lines of the file:
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@@
 		(layer "Edge.Cuts")
+	)
+	(gr_text "PIN 1"
+		(at 121 76.31 0)
+		(layer "F.SilkS")
+		(effects
+			(font
+				(size 0.7 0.7)
+				(thickness 0.15)
+			)
+		)
 	)
 	(gr_text "r l"
@@
 			)
 		)
+	)
+	(gr_text "3V3 REG"
+		(at 72 76.375 0)
+		(layer "F.SilkS")
+		(effects
+			(font
+				(size 0.8 0.8)
+				(thickness 0.15)
+			)
+		)
+	)
+	(gr_text "PSM712"
+		(at 79.5 48.105 0)
+		(layer "F.SilkS")
+		(effects
+			(font
+				(size 0.8 0.8)
+				(thickness 0.15)
+			)
+		)
+	)
+	(gr_text "TLV9062"
+		(at 80 55.605 0)
+		(layer "F.SilkS")
+		(effects
+			(font
+				(size 0.8 0.8)
+				(thickness 0.15)
+			)
+		)
+	)
+	(gr_text "B5819"
+		(at 84 82.405 0)
+		(layer "F.SilkS")
+		(effects
+			(font
+				(size 0.8 0.8)
+				(thickness 0.15)
+			)
+		)
+	)
+	(gr_text "PTC"
+		(at 88.25 81.274999 0)
+		(layer "F.SilkS")
+		(effects
+			(font
+				(size 0.8 0.8)
+				(thickness 0.15)
+			)
+		)
+	)
+	(gr_text "ISO7741"
+		(at 98.5 70.5 0)
+		(layer "F.SilkS")
+		(effects
+			(font
+				(size 0.8 0.8)
+				(thickness 0.15)
+			)
+		)
+	)
+	(gr_text "AIC3204"
+		(at 100 41.925 0)
+		(layer "F.SilkS")
+		(effects
+			(font
+				(size 0.8 0.8)
+				(thickness 0.15)
+			)
+		)
+	)
+	(gr_text "ISO1540"
+		(at 108.5 65.854999 0)
+		(layer "F.SilkS")
+		(effects
+			(font
+				(size 0.8 0.8)
+				(thickness 0.15)
+			)
+		)
+	)
+	(gr_text "5V REG"
+		(at 79 79 90)
+		(layer "F.SilkS")
+		(effects
+			(font
+				(size 0.8 0.8)
+				(thickness 0.15)
+			)
+		)
+	)
+	(gr_text "TLV9062"
+		(at 104.155 48.5 90)
+		(layer "F.SilkS")
+		(effects
+			(font
+				(size 0.8 0.8)
+				(thickness 0.15)
+			)
+		)
+	)
+	(gr_text "TPA6139"
+		(at 107.205 42 90)
+		(layer "F.SilkS")
+		(effects
+			(font
+				(size 0.8 0.8)
+				(thickness 0.15)
+			)
+		)
+	)
+	(gr_text "B0505S"
+		(at 130.544999 70.5 90)
+		(layer "F.SilkS")
+		(effects
+			(font
+				(size 0.8 0.8)
+				(thickness 0.15)
+			)
+		)

Commit message: Analog leveller on the carrier board (LED/LDR vactrols, MCP4725, TLV9062), fx loop left open, simulated
Co-Authored-By: Claude Opus 5.5 <noreply@anthropic.com>
Parts:
- added C80: 10uF, C_0402_1005Metric, F.Cu at (92.8, 35.5)
- added C82: 100nF, C_0402_1005Metric, F.Cu at (89.5, 55.8)
- added C83: 100nF, C_0402_1005Metric, F.Cu at (89.8, 43.2)
- added C85: 10uF, C_0402_1005Metric, F.Cu at (77.5, 34.5)
- added OC1: LED+LDR, OPTO_PAIR_LED3_LDR5, B.Cu at (83.8, 40.8)
- added OC2: LED+LDR, OPTO_PAIR_LED3_LDR5, B.Cu at (80.5, 41.2)
- added Q1: MMBT3904, SOT-23, F.Cu at (78.2, 38.0)
- added R80: 4.7k, R_0402_1005Metric, F.Cu at (92.8, 43.5)
- added R81: 100k, R_0402_1005Metric, F.Cu at (92.5, 45.5)
- added R82: 1k, R_0402_1005Metric, F.Cu at (81.2, 37.0)
- added R83: 100, R_0402_1005Metric, F.Cu at (79.2, 34.8)
- added R85: 4.7k, R_0402_1005Metric, F.Cu at (89.0, 38.0)
- added R86: 100k, R_0402_1005Metric, F.Cu at (81.0, 34.5)
- added U15: MCP4725, SOT-23-6, F.Cu at (89.5, 53.0)
- added U16: TLV9062, Texas_DSG0008A_WSON-8-1EP_2x2mm_P0.5mm_EP0.9x1.6mm, F.Cu at (89.8, 40.8)
Routing:
- net FXR_R: track 16.0 -> 68.6 mm, vias 1 -> 3
- net ISO5V_RAW: track 28.3 -> 76.6 mm, vias 2 -> 4
- net ISDA: track 56.9 -> 89.6 mm, vias 3 -> 5
- net FXR_L: track 17.2 -> 48.1 mm, vias 1 -> 3
- net LO_L: track 20.6 -> 51.2 mm, vias 1 -> 5
- net LO_R: track 23.2 -> 52.7 mm, vias 1 -> 3
- net ISO3V3: track 127.8 -> 156.0 mm, vias 5 -> 6
- net LED_DAC: track 0.00 -> 23.0 mm, vias 0 -> 2
- net IGND: track 314.6 -> 330.9 mm
- net LVC_L: track 0.00 -> 16.0 mm, vias 0 -> 2
- net ISO5V: track 79.2 -> 93.5 mm, vias 6 -> 8
- net LVA_R: track 0.00 -> 13.8 mm, vias 0 -> 2
- net ISCL: track 58.3 -> 67.0 mm, vias 3 -> 6
- net LVA_L: track 0.00 -> 7.12 mm
- net LVC_R: track 0.00 -> 5.72 mm
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Other:
- board text added: "3904"
- board text added: "MCP4725"

Commit message: Power switch, re-centred header holes, input headroom + ADC range + power-on thump fixes found by scenario simulation
Co-Authored-By: Claude Opus 5.5 <noreply@anthropic.com>
Parts:
- added D63: 1N4148WS, D_SOD-323, F.Cu at (113.5, 32.5)
- R33, R43: value 1M -> 470k
- R34, R44: value 20k -> 4.7k
- R70: value 470k -> 1M
Routing:
- net HP_ON: track 9.63 -> 19.0 mm, vias 0 -> 2
- net ISO3V3: track 156.0 -> 164.7 mm
Other:
- board text added: "in gain knob"
- board text added: "out gain knob"
- board text removed: "pg-hp"
- board text removed: "pg-line"

Commit message: Hard input clamp and output ceiling, guitar-friendly input, firmware codec guard; black chicken heads for power + page (measured sweeps), 9 V jack in the left wall
Co-Authored-By: Claude Opus 5.5 <noreply@anthropic.com>
Parts:
- R34, R44: value 4.7k -> 20k
- R6: value 10k -> 3.3k
Changed lines of the file:
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@@
 			)
 		)
-		(property "Value" "4.7k"
+		(property "Value" "20k"
 			(at 0 1.17 0)
 			(layer "F.Fab")
@@
 			)
 		)
-		(property "Value" "10k"
+		(property "Value" "3.3k"
 			(at 0 1.17 90)
 			(layer "F.Fab")
@@
 			)
 		)
-		(property "Value" "4.7k"
+		(property "Value" "20k"
 			(at 0 1.17 0)
 			(layer "F.Fab")

Commit message: 47 ohm headphone power cap, power dial ON zone, wiring pictures
Co-Authored-By: Claude Opus 5.5 <noreply@anthropic.com>
Parts:
- R50, R60: value 1 -> 47
Changed lines of the file:
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@@
 			)
 		)
-		(property "Value" "1"
+		(property "Value" "47"
 			(at 0 1.43 90)
 			(layer "F.Fab")
@@
 			)
 		)
-		(property "Value" "1"
+		(property "Value" "47"
 			(at 0 1.43 0)
 			(layer "F.Fab")
